Commit message: use xacro definitions for urdfs

File: urdf/oc110.urdf.xacro (robot description, xacro)
@@ -1,29 +1,35 @@
 <?xml version="1.0"?>
 <robot name="wibotic_oc110" xmlns:xacro="http://ros.org/wiki/xacro">
-  <link name="charger_frame"/>
-  <joint name="oc110_joint" type="fixed">
-    <origin xyz="$(arg px) $(arg py) $(arg pz)" rpy="$(arg or) $(arg op) $(arg oy)"/>
-    <parent link="charger_frame"/>
-    <child link="charger_link"/>
-  </joint>
-  <link name="charger_link">
-    <collision name="collision">
-      <geometry>
-        <mesh filename="../meshes/OC110.dae"/>
-      </geometry>
-    </collision>
-    <visual name="visual">
-      <geometry>
-        <mesh filename="../meshes/OC110.dae"/>
-      </geometry>
-    </visual>
-    <inertial>
-      <mass value="0.1"/>
-      <origin xyz="0 0 0"/>
-      <inertia ixx="0.00001887" ixy="0.0" ixz="0.0"
-               iyy="0.00001887" iyz="0.0"
-               izz="0.00001887"/>
-    </inertial>
-  </link>
-  <wibotic_sim_oc110/>
+  <xacro:macro name="wibotic_oc110" params="parent p_x:=0 p_y:=0 p_z:=0 o_r:=0 o_p:=0 o_y:=0">
+    <joint name="oc110_joint1" type="fixed">
+      <origin xyz="${p_x} ${p_y} ${p_z}" rpy="${o_r} ${o_p} ${o_y}"/>
+      <parent link="${parent}"/>
+      <child link="charger_frame"/>
+    </joint>
+    <link name="charger_frame"/>
+    <joint name="oc110_joint2" type="fixed">
+      <parent link="charger_frame"/>
+      <child link="charger_link"/>
+    </joint>
+    <link name="charger_link">
+      <collision name="collision">
+        <geometry>
+          <mesh filename="package://wibotic_models/meshes/OC110.dae"/>
+        </geometry>
+      </collision>
+      <visual name="visual">
+        <geometry>
+          <mesh filename="package://wibotic_models/meshes/OC110.dae"/>
+        </geometry>
+      </visual>
+      <inertial>
+        <mass value="0.1"/>
+        <origin xyz="0 0 0"/>
+        <inertia ixx="0.00001887" ixy="0.0" ixz="0.0"
+                 iyy="0.00001887" iyz="0.0"
+                 izz="0.00001887"/>
+      </inertial>
+    </link>
+    <wibotic_sim_oc110/>
+  </xacro:macro>
 </robot>

File: urdf/oc210.urdf.xacro (robot description, xacro)
@@ -1,29 +1,35 @@
 <?xml version="1.0"?>
 <robot name="wibotic_oc210" xmlns:xacro="http://ros.org/wiki/xacro">
-  <link name="charger_frame"/>
-  <joint name="oc210_joint" type="fixed">
-    <origin xyz="$(arg px) $(arg py) $(arg pz)" rpy="$(arg or) $(arg op) $(arg oy)"/>
-    <parent link="charger_frame"/>
-    <child link="charger_link"/>
-  </joint>
-  <link name="charger_link">
-    <collision name="collision">
-      <geometry>
-        <mesh filename="../meshes/OC210.dae"/>
-      </geometry>
-    </collision>
-    <visual name="visual">
-      <geometry>
-        <mesh filename="../meshes/OC210.dae"/>
-      </geometry>
-    </visual>
-    <inertial>
-      <mass value="0.1"/>
-      <origin xyz="0 0 0"/>
-      <inertia ixx="0.00001887" ixy="0.0" ixz="0.0"
-               iyy="0.00001887" iyz="0.0"
-               izz="0.00001887"/>
-    </inertial>
-  </link>
-  <wibotic_sim_oc210/>
+  <xacro:macro name="wibotic_oc210" params="parent p_x:=0 p_y:=0 p_z:=0 o_r:=0 o_p:=0 o_y:=0">
+    <joint name="oc210_joint1" type="fixed">
+      <origin xyz="${p_x} ${p_y} ${p_z}" rpy="${o_r} ${o_p} ${o_y}"/>
+      <parent link="${parent}"/>
+      <child link="charger_frame"/>
+    </joint>
+    <link name="charger_frame"/>
+    <joint name="oc210_joint2" type="fixed">
+      <parent link="charger_frame"/>
+      <child link="charger_link"/>
+    </joint>
+    <link name="charger_link">
+      <collision name="collision">
+        <geometry>
+          <mesh filename="package://wibotic_models/meshes/OC210.dae"/>
+        </geometry>
+      </collision>
+      <visual name="visual">
+        <geometry>
+          <mesh filename="package://wibotic_models/meshes/OC210.dae"/>
+        </geometry>
+      </visual>
+      <inertial>
+        <mass value="0.1"/>
+        <origin xyz="0 0 0"/>
+        <inertia ixx="0.00001887" ixy="0.0" ixz="0.0"
+                 iyy="0.00001887" iyz="0.0"
+                 izz="0.00001887"/>
+      </inertial>
+    </link>
+    <wibotic_sim_oc210/>
+  </xacro:macro>
 </robot>

File: urdf/oc250.urdf.xacro (robot description, xacro)
@@ -1,29 +1,35 @@
 <?xml version="1.0"?>
 <robot name="wibotic_oc250" xmlns:xacro="http://ros.org/wiki/xacro">
-  <link name="charger_frame"/>
-  <joint name="oc250_joint" type="fixed">
-    <origin xyz="$(arg px) $(arg py) $(arg pz)" rpy="$(arg or) $(arg op) $(arg oy)"/>
-    <parent link="charger_frame"/>
-    <child link="charger_link"/>
-  </joint>
-  <link name="charger_link">
-    <collision name="collision">
-      <geometry>
-        <mesh filename="../meshes/OC250.dae"/>
-      </geometry>
-    </collision>
-    <visual name="visual">
-      <geometry>
-        <mesh filename="../meshes/OC250.dae"/>
-      </geometry>
-    </visual>
-    <inertial>
-      <mass value="0.1"/>
-      <origin xyz="0 0 0"/>
-      <inertia ixx="0.00001887" ixy="0.0" ixz="0.0"
-               iyy="0.00001887" iyz="0.0"
-               izz="0.00001887"/>
-    </inertial>
-  </link>
-  <wibotic_sim_oc250/>
+  <xacro:macro name="wibotic_oc250" params="parent p_x:=0 p_y:=0 p_z:=0 o_r:=0 o_p:=0 o_y:=0">
+    <joint name="oc250_joint1" type="fixed">
+      <origin xyz="${p_x} ${p_y} ${p_z}" rpy="${o_r} ${o_p} ${o_y}"/>
+      <parent link="${parent}"/>
+      <child link="charger_frame"/>
+    </joint>
+    <link name="charger_frame"/>
+    <joint name="oc250_joint2" type="fixed">
+      <parent link="charger_frame"/>
+      <child link="charger_link"/>
+    </joint>
+    <link name="charger_link">
+      <collision name="collision">
+        <geometry>
+          <mesh filename="package://wibotic_models/meshes/OC250.dae"/>
+        </geometry>
+      </collision>
+      <visual name="visual">
+        <geometry>
+          <mesh filename="package://wibotic_models/meshes/OC250.dae"/>
+        </geometry>
+      </visual>
+      <inertial>
+        <mass value="0.1"/>
+        <origin xyz="0 0 0"/>
+        <inertia ixx="0.00001887" ixy="0.0" ixz="0.0"
+                 iyy="0.00001887" iyz="0.0"
+                 izz="0.00001887"/>
+      </inertial>
+    </link>
+    <wibotic_sim_oc250/>
+  </xacro:macro>
 </robot>

File: urdf/oc300.urdf.xacro (robot description, xacro)
@@ -1,29 +1,35 @@
 <?xml version="1.0"?>
 <robot name="wibotic_oc300" xmlns:xacro="http://ros.org/wiki/xacro">
-  <link name="charger_frame"/>
-  <joint name="oc300_joint" type="fixed">
-    <origin xyz="$(arg px) $(arg py) $(arg pz)" rpy="$(arg or) $(arg op) $(arg oy)"/>
-    <parent link="charger_frame"/>
-    <child link="charger_link"/>
-  </joint>
-  <link name="charger_link">
-    <collision name="collision">
-      <geometry>
-        <mesh filename="../meshes/OC300.dae"/>
-      </geometry>
-    </collision>
-    <visual name="visual">
-      <geometry>
-        <mesh filename="../meshes/OC300.dae"/>
-      </geometry>
-    </visual>
-    <inertial>
-      <mass value="0.1"/>
-      <origin xyz="0 0 0"/>
-      <inertia ixx="0.00001887" ixy="0.0" ixz="0.0"
-               iyy="0.00001887" iyz="0.0"
-               izz="0.00001887"/>
-    </inertial>
-  </link>
-  <wibotic_sim_oc300/>
+  <xacro:macro name="wibotic_oc300" params="parent p_x:=0 p_y:=0 p_z:=0 o_r:=0 o_p:=0 o_y:=0">
+    <joint name="oc300_joint1" type="fixed">
+      <origin xyz="${p_x} ${p_y} ${p_z}" rpy="${o_r} ${o_p} ${o_y}"/>
+      <parent link="${parent}"/>
+      <child link="charger_frame"/>
+    </joint>
+    <link name="charger_frame"/>
+    <joint name="oc300_joint2" type="fixed">
+      <parent link="charger_frame"/>
+      <child link="charger_link"/>
+    </joint>
+    <link name="charger_link">
+      <collision name="collision">
+        <geometry>
+          <mesh filename="package://wibotic_models/meshes/OC300.dae"/>
+        </geometry>
+      </collision>
+      <visual name="visual">
+        <geometry>
+          <mesh filename="package://wibotic_models/meshes/OC300.dae"/>
+        </geometry>
+      </visual>
+      <inertial>
+        <mass value="0.1"/>
+        <origin xyz="0 0 0"/>
+        <inertia ixx="0.00001887" ixy="0.0" ixz="0.0"
+                 iyy="0.00001887" iyz="0.0"
+                 izz="0.00001887"/>
+      </inertial>
+    </link>
+    <wibotic_sim_oc300/>
+  </xacro:macro>
 </robot>

File: urdf/rc100.urdf.xacro (robot description, xacro)
@@ -1,7 +1,12 @@
 <?xml version="1.0"?>
 <robot name="wibotic_rc100" xmlns:xacro="http://ros.org/wiki/xacro">
+  <xacro:macro name="wibotic_rc100" params="parent p_x:=0 p_y:=0 p_z:=0 o_r:=0 o_p:=0 o_y:=0">
     <link name="coil_frame"/>
     <joint name="rc100_joint1" type="fixed">
-      <origin xyz="$(arg px) $(arg py) $(arg pz)" rpy="$(arg or) $(arg op) $(arg oy)"/>
+      <origin xyz="${p_x} ${p_y} ${p_z}" rpy="${o_r} ${o_p} ${o_y}"/>
+      <parent link="${parent}"/>
+      <child link="coil_frame"/>
+    </joint>
+    <joint name="rc100_joint2" type="fixed">
       <parent link="coil_frame"/>
       <child link="coil_link"/>
@@ -10,10 +15,16 @@
       <collision name="collision">
         <geometry>
-          <mesh filename="../meshes/RC100.dae"/>
+          <mesh filename="package://wibotic_models/meshes/RC100.dae"/>
+        </geometry>
+      </collision>
+      <collision name="COIL_CENTER">
+        <origin xyz="0.0545 0.00605 0.0565" rpy="0 0 0"/>
+        <geometry>
+          <sphere radius="0.001"/>
         </geometry>
       </collision>
       <visual name="visual">
         <geometry>
-          <mesh filename="../meshes/RC100.dae"/>
+          <mesh filename="package://wibotic_models/meshes/RC100.dae"/>
         </geometry>
       </visual>
@@ -28,3 +39,4 @@
     </link>
     <wibotic_sim_rc100/>
+  </xacro:macro>
 </robot>

File: urdf/tc200.urdf.xacro (robot description, xacro)
@@ -1,7 +1,12 @@
 <?xml version="1.0"?>
 <robot name="wibotic_tc200" xmlns:xacro="http://ros.org/wiki/xacro">
+  <xacro:macro name="wibotic_tc200" params="parent p_x:=0 p_y:=0 p_z:=0 o_r:=0 o_p:=0 o_y:=0">
     <link name="coil_frame"/>
     <joint name="tc200_joint1" type="fixed">
-      <origin xyz="$(arg px) $(arg py) $(arg pz)" rpy="$(arg or) $(arg op) $(arg oy)"/>
+      <origin xyz="${p_x} ${p_y} ${p_z}" rpy="${o_r} ${o_p} ${o_y}"/>
+      <parent link="${parent}"/>
+      <child link="coil_frame"/>
+    </joint>
+    <joint name="tc200_joint2" type="fixed">
       <parent link="coil_frame"/>
       <child link="coil_link"/>
@@ -10,10 +15,16 @@
       <collision name="collision">
         <geometry>
-          <mesh filename="../meshes/TC200.dae"/>
+          <mesh filename="package://wibotic_models/meshes/TC200.dae"/>
+        </geometry>
+      </collision>
+      <collision name="COIL_CENTER">
+        <origin xyz="0.105 0.01 0.107" rpy="0 0 0"/>
+        <geometry>
+          <sphere radius="0.001"/>
         </geometry>
       </collision>
       <visual name="visual">
         <geometry>
-          <mesh filename="../meshes/TC200.dae"/>
+          <mesh filename="package://wibotic_models/meshes/TC200.dae"/>
         </geometry>
       </visual>
@@ -28,3 +39,4 @@
     </link>
     <wibotic_sim_tc200/>
+  </xacro:macro>
 </robot>

File: urdf/tr100.urdf.xacro (robot description, xacro)
@@ -1,29 +1,31 @@
 <?xml version="1.0"?>
 <robot name="wibotic_tr100" xmlns:xacro="http://ros.org/wiki/xacro">
-  <link name="transmitter_frame"/>
-  <joint name="tr100_joint" type="fixed">
-    <origin xyz="$(arg px) $(arg py) $(arg pz)" rpy="$(arg or) $(arg op) $(arg oy)"/>
-    <parent link="transmitter_frame"/>
-    <child link="transmitter_link"/>
-  </joint>
-  <link name="transmitter_link">
-    <collision name="collision">
-      <geometry>
-        <mesh filename="../meshes/TR100.dae"/>
-      </geometry>
-    </collision>
-    <visual name="visual">
-      <geometry>
-        <mesh filename="../meshes/TR100.dae"/>
-      </geometry>
-    </visual>
-    <inertial>
-      <mass value="0.1"/>
-      <origin xyz="0 0 0"/>
-      <inertia ixx="0.00001887" ixy="0.0" ixz="0.0"
-               iyy="0.00001887" iyz="0.0"
-               izz="0.00001887"/>
-    </inertial>
-  </link>
-  <wibotic_sim_tr100/>
+  <xacro:macro name="wibotic_tr100" params="parent p_x:=0 p_y:=0 p_z:=0 o_r:=0 o_p:=0 o_y:=0">
+    <link name="transmitter_frame"/>
+    <joint name="tr100_joint" type="fixed">
+      <origin xyz="${p_x} ${p_y} ${p_z}" rpy="${o_r} ${o_p} ${o_y}"/>
+      <parent link="transmitter_frame"/>
+      <child link="transmitter_link"/>
+    </joint>
+    <link name="transmitter_link">
+      <collision name="collision">
+        <geometry>
+          <mesh filename="package://wibotic_models/meshes/TR100.dae"/>
+        </geometry>
+      </collision>
+      <visual name="visual">
+        <geometry>
+          <mesh filename="package://wibotic_models/meshes/TR100.dae"/>
+        </geometry>
+      </visual>
+      <inertial>
+        <mass value="0.1"/>
+        <origin xyz="0 0 0"/>
+        <inertia ixx="0.00001887" ixy="0.0" ixz="0.0"
+                 iyy="0.00001887" iyz="0.0"
+                 izz="0.00001887"/>
+      </inertial>
+    </link>
+    <wibotic_sim_tr100/>
+  </xacro:macro>
 </robot>

File: urdf/tr300.urdf.xacro (robot description, xacro)
@@ -1,29 +1,31 @@
 <?xml version="1.0"?>
 <robot name="wibotic_tr300" xmlns:xacro="http://ros.org/wiki/xacro">
-  <link name="transmitter_frame"/>
-  <joint name="tr300_joint" type="fixed">
-    <origin xyz="$(arg px) $(arg py) $(arg pz)" rpy="$(arg or) $(arg op) $(arg oy)"/>
-    <parent link="transmitter_frame"/>
-    <child link="transmitter_link"/>
-  </joint>
-  <link name="transmitter_link">
-    <collision name="collision">
-      <geometry>
-        <mesh filename="../meshes/TR300.dae"/>
-      </geometry>
-    </collision>
-    <visual name="visual">
-      <geometry>
-        <mesh filename="../meshes/TR300.dae"/>
-      </geometry>
-    </visual>
-    <inertial>
-      <mass value="0.1"/>
-      <origin xyz="0 0 0"/>
-      <inertia ixx="0.00001887" ixy="0.0" ixz="0.0"
-               iyy="0.00001887" iyz="0.0"
-               izz="0.00001887"/>
-    </inertial>
-  </link>
-  <wibotic_sim_tr300/>
+  <xacro:macro name="wibotic_tr300" params="parent p_x:=0 p_y:=0 p_z:=0 o_r:=0 o_p:=0 o_y:=0">
+    <link name="transmitter_frame"/>
+    <joint name="tr300_joint" type="fixed">
+      <origin xyz="${p_x} ${p_y} ${p_z}" rpy="${o_r} ${o_p} ${o_y}"/>
+      <parent link="transmitter_frame"/>
+      <child link="transmitter_link"/>
+    </joint>
+    <link name="transmitter_link">
+      <collision name="collision">
+        <geometry>
+          <mesh filename="package://wibotic_models/meshes/TR300.dae"/>
+        </geometry>
+      </collision>
+      <visual name="visual">
+        <geometry>
+          <mesh filename="package://wibotic_models/meshes/TR300.dae"/>
+        </geometry>
+      </visual>
+      <inertial>
+        <mass value="0.1"/>
+        <origin xyz="0 0 0"/>
+        <inertia ixx="0.00001887" ixy="0.0" ixz="0.0"
+                 iyy="0.00001887" iyz="0.0"
+                 izz="0.00001887"/>
+      </inertial>
+    </link>
+    <wibotic_sim_tr300/>
+  </xacro:macro>
 </robot>
