Commit message: update urdf, add launch files and robots

File: urdf/rc100.urdf.xacro (robot description, xacro)
@@ -38,4 +38,9 @@
       </inertial>
     </link>
+    <gazebo>
+      <plugin name="rx_plugin" filename="libwibotic_coil_plugin.so">
+        <coilType>receive</coilType>
+      </plugin>
+    </gazebo>
     <wibotic_sim_rc100/>
   </xacro:macro>

File: urdf/tc200.urdf.xacro (robot description, xacro)
@@ -38,4 +38,9 @@
       </inertial>
     </link>
+    <gazebo>
+      <plugin name="tx_plugin" filename="libwibotic_coil_plugin.so">
+        <coilType>transmit</coilType>
+      </plugin>
+    </gazebo>
     <wibotic_sim_tc200/>
   </xacro:macro>

File: urdf/tr110.urdf.xacro (robot description, xacro)
@@ -1,7 +1,12 @@
 <?xml version="1.0"?>
-<robot name="wibotic_tr100" xmlns:xacro="http://ros.org/wiki/xacro">
-  <xacro:macro name="wibotic_tr100" params="parent p_x:=0 p_y:=0 p_z:=0 o_r:=0 o_p:=0 o_y:=0">
+<robot name="wibotic_tr110" xmlns:xacro="http://ros.org/wiki/xacro">
+  <xacro:macro name="wibotic_tr110" params="parent p_x:=0 p_y:=0 p_z:=0 o_r:=0 o_p:=0 o_y:=0">
     <link name="transmitter_frame"/>
-    <joint name="tr100_joint" type="fixed">
+    <joint name="tr110_joint_1" type="fixed">
+      <origin xyz="${p_x} ${p_y} ${p_z}" rpy="${o_r} ${o_p} ${o_y}"/>
+      <parent link="${parent}"/>
+      <child link="transmitter_frame"/>
+    </joint>
+    <joint name="tr110_joint_2" type="fixed">
       <origin xyz="${p_x} ${p_y} ${p_z}" rpy="${o_r} ${o_p} ${o_y}"/>
       <parent link="transmitter_frame"/>
@@ -27,5 +32,5 @@
       </inertial>
     </link>
-    <wibotic_sim_tr100/>
+    <wibotic_sim_tr110/>
   </xacro:macro>
 </robot>

File: urdf/tr300.urdf.xacro (robot description, xacro)
@@ -3,5 +3,10 @@
   <xacro:macro name="wibotic_tr300" params="parent p_x:=0 p_y:=0 p_z:=0 o_r:=0 o_p:=0 o_y:=0">
     <link name="transmitter_frame"/>
-    <joint name="tr300_joint" type="fixed">
+    <joint name="tr300_joint_1" type="fixed">
+      <origin xyz="${p_x} ${p_y} ${p_z}" rpy="${o_r} ${o_p} ${o_y}"/>
+      <parent link="${parent}"/>
+      <child link="transmitter_frame"/>
+    </joint>
+    <joint name="tr300_joint_2" type="fixed">
       <origin xyz="${p_x} ${p_y} ${p_z}" rpy="${o_r} ${o_p} ${o_y}"/>
       <parent link="transmitter_frame"/>
